Commit message: Updates

File: General/notes/resource/kuka_iiwa.urdf (robot description, URDF)
Before this commit: robot lbr_iiwa, 8 links, 7 joints
Links:
- added link tool0, mass 1.0; visual mesh filename=meshes/link_7.obj
Joints:
- added joint tool_joint: type fixed, parent lbr_iiwa_link_7, child tool0, origin xyz=0 0 0.5 rpy=0 0 0

Commit message: Updates

File: General/notes/resource/kuka_iiwa.urdf (robot description, URDF)
Before this commit: robot lbr_iiwa, 9 links, 8 joints
Links:
- link tool0: geometry collision box size=0.1 0.2 0.72; visual box size=0.1 0.2 0.72
Joints:
- joint tool_joint: origin xyz=0 0 0.5 rpy=0 0 0 -> xyz=0 0 0 rpy=0 0 0

Commit message: Updates to urdf

File: General/notes/resource/kuka_iiwa.urdf (robot description, URDF)
Before this commit: robot lbr_iiwa, 9 links, 8 joints
Links:
- removed link tool0
Joints:
- removed joint tool_joint
