Commit message: Updated urdf

File: General/notes/resource/kuka_iiwa_payload.urdf (robot description, URDF)
Before this commit: robot lbr_iiwa, 8 links, 7 joints
Links:
- added link tool0, mass 1.0; collision box size=0.1 0.1 0.1; visual box size=0.1 0.1 0.1
Joints:
- added joint tool_joint: type fixed, parent lbr_iiwa_link_7, child tool0, origin xyz=0 0 0 rpy=0 0 0
