Commit message: Actuator bandwidth

File: General/notes/resource/kuka_iiwa_offset.urdf (robot description, URDF)
Before this commit: robot lbr_iiwa, 8 links, 7 joints
Joints:
- joint lbr_iiwa_joint_7: origin xyz=0 0.0 0 rpy=-1.57079632679 3.14159265359 0 -> xyz=0.12 0.0 0.1 rpy=-1.57079632679 3.14159265359 0
