Commit message: fixed joint

File: General/notes/resource/two_dof.urdf (robot description, URDF)
Before this commit: robot TwoJointRobot, 3 links, 2 joints
Links:
- added link ee_ball, mass 10; collision sphere radius=0.1; visual sphere radius=0.1
- added link flange, mass 0.0000; collision box size=0.001 0.001 0.001; visual box size=0.001 0.001 0.001
Joints:
- added joint ee_ball: type fixed, parent flange, child ee_ball, origin xyz=1 0 0 rpy=0 0 0, axis 0 0 1, limit lower=-3.01069 upper=3.01069 effort=12 velocity=2.6100
- added joint flange_joint: type fixed, parent link_2, child flange, origin xyz=0 0 0 rpy=0 0 0, axis 0 0 1
